File: jacdac_access_switch_interface.kicad_sch (KiCad schematic)
At the start: 42 parts

Commit message: v1.7 complete and sent for manufacture
Parts:
- U: LCSC C52923 -> C1525
- U: LCSC C457666 -> C457666
- U: LCSC C60490 -> C25744
- U: LCSC C270649 -> C25082
- U: LCSC C25105 -> C25104
- U: LCSC C25756 -> C25082
Connections:
- net JD_STATUS: now also U.1 (PB7/PB8)
- no-connect marks 2 -> 1
Changed lines of the file:
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@@
   (junction (at 44.45 40.64) (diameter 0) (color 0 0 0 0)
   )
-  (no_connect (at 50.8 153.67))
   (no_connect (at 50.8 158.75))
   (wire (pts (xy 91.44 163.83) (xy 102.87 163.83))
@@
     (stroke (width 0) (type default))
   )
+  (wire (pts (xy 50.8 153.67) (xy 40.64 153.67))
+    (stroke (width 0) (type default))
+  )
   (wire (pts (xy 76.2 105.41) (xy 76.2 100.33))
     (stroke (width 0) (type default))
@@
   )
   (label "RING1_P" (at 226.06 91.44 0) (fields_autoplaced)
+    (effects (font (size 1.27 1.27)) (justify left bottom))
+  )
+  (label "JD_STATUS" (at 40.64 153.67 0) (fields_autoplaced)
     (effects (font (size 1.27 1.27)) (justify left bottom))
   )
@@
     (pin "1")
   )
-  (symbol (lib_id "Device:D_TVS") (at 44.45 58.42 270) (unit 1)
-    (in_bom yes) (on_board yes)
-    (default_instance (reference "U") (unit 1) (value "") (footprint ""))
-    (property "Reference" "U" (id 0) (at 39.37 58.42 90)
-      (effects (font (size 1.27 1.27)) (justify left))
-    )
-    (property "Value" "" (id 1) (at 25.4 60.96 90)
+  (symbol (lib_name "D_TVS_1") (lib_id "Device:D_TVS") (at 44.45 58.42 270) (unit 1)
+    (in_bom yes) (on_board yes)
+    (default_instance (reference "U") (unit 1) (value "") (footprint ""))
+    (property "Reference" "U" (id 0) (at 39.37 60.96 90)
+      (effects (font (size 1.27 1.27)) (justify left))
+    )
+    (property "Value" "" (id 1) (at 26.67 58.42 90)
       (effects (font (size 1.27 1.27)) (justify left))
     )
@@
       (effects (font (size 1.27 1.27)) (justify left))
     )
-    (property "Value" "" (id 1) (at 59.69 52.07 0)
+    (property "Value" "" (id 1) (at 66.04 55.88 90)
       (effects (font (size 1.27 1.27)) (justify left))
     )
@@
       (effects (font (size 1.27 1.27)) hide)
     )
-    (property "LCSC" "C52923" (id 4) (at 40.64 185.42 0)
+    (property "LCSC" "C1525" (id 4) (at 40.64 185.42 0)
       (effects (font (size 1.27 1.27)) hide)
     )
@@
       (effects (font (size 1.27 1.27)) hide)
     )
-    (property "LCSC" "C457666 " (id 4) (at 63.5 106.68 0)
+    (property "LCSC" "C457666" (id 4) (at 63.5 106.68 0)
       (effects (font (size 1.27 1.27)) hide)
     )
@@
       (effects (font (size 1.27 1.27)) hide)
     )
-    (property "LCSC" "C60490" (id 4) (at 209.55 63.5 90)
+    (property "LCSC" "C25744" (id 4) (at 209.55 63.5 90)
       (effects (font (size 1.27 1.27)) hide)
     )
@@
       (effects (font (size 1.27 1.27)) hide)
     )
-    (property "LCSC" "C60490" (id 4) (at 209.55 91.44 90)
+    (property "LCSC" "C25744" (id 4) (at 209.55 91.44 90)
       (effects (font (size 1.27 1.27)) hide)
     )
@@
       (effects (font (size 1.27 1.27)) hide)
     )
-    (property "LCSC" "C270649" (id 4) (at 109.22 80.01 90)
+    (property "LCSC" "C25082" (id 4) (at 109.22 80.01 90)
       (effects (font (size 1.27 1.27)) hide)
     )
@@
     (pin "1")
   )
-  (symbol (lib_name "jack_3.5mm_PJ313D_1") (lib_id "jacdac_access_switch_interface:jack_3.5mm_PJ313D") (at 138.43 30.48 0) (unit 1)
+  (symbol (lib_id "jacdac_access_switch_interface:jack_3.5mm_PJ313D") (at 138.43 30.48 0) (unit 1)
     (in_bom yes) (on_board yes)
     (default_instance (reference "J") (unit 1) (value "jack_3.5_pj313d") (footprint "jacdac_access_switch_interface:jack_3.5_pj313d_smt"))
@@
       (effects (font (size 1.27 1.27)) hide)
     )
-    (property "LCSC" "C25105" (id 4) (at 227.33 151.13 90)
+    (property "LCSC" "C25104" (id 4) (at 227.33 151.13 90)
       (effects (font (size 1.27 1.27)) hide)
     )
@@
       (effects (font (size 1.27 1.27)) hide)
     )
-    (property "LCSC" "C60490" (id 4) (at 255.27 91.44 90)
+    (property "LCSC" "C25744" (id 4) (at 255.27 91.44 90)
       (effects (font (size 1.27 1.27)) hide)
     )
@@
       (effects (font (size 1.27 1.27)) hide)
     )
-    (property "LCSC" "C60490" (id 4) (at 209.55 35.56 90)
+    (property "LCSC" "C25744" (id 4) (at 209.55 35.56 90)
       (effects (font (size 1.27 1.27)) hide)
     )
@@
       (effects (font (size 1.27 1.27)) hide)
     )
-    (property "LCSC" "C25756 " (id 4) (at 151.13 73.66 90)
+    (property "LCSC" "C25082" (id 4) (at 151.13 73.66 90)
       (effects (font (size 1.27 1.27)) hide)
     )
@@
       (effects (font (size 1.27 1.27)) hide)
     )
-    (property "LCSC" "C60490" (id 4) (at 255.27 63.5 90)
+    (property "LCSC" "C25744" (id 4) (at 255.27 63.5 90)
       (effects (font (size 1.27 1.27)) hide)
     )
@@
       (effects (font (size 1.27 1.27)) hide)
     )
-    (property "LCSC" "C60490" (id 4) (at 255.27 35.56 90)
+    (property "LCSC" "C25744" (id 4) (at 255.27 35.56 90)
       (effects (font (size 1.27 1.27)) hide)
     )
@@
       (effects (font (size 1.27 1.27)) hide)
     )
-    (property "LCSC" "C25105" (id 4) (at 228.6 130.81 90)
+    (property "LCSC" "C25104" (id 4) (at 228.6 130.81 90)
       (effects (font (size 1.27 1.27)) hide)
     )
@@
     (pin "3")
   )
-  (symbol (lib_name "TLP240A_1") (lib_id "jacdac_access_switch_interface:TLP240A") (at 240.03 133.35 0) (unit 1)
+  (symbol (lib_id "jacdac_access_switch_interface:TLP240A") (at 240.03 133.35 0) (unit 1)
     (in_bom yes) (on_board yes) (fields_autoplaced)
     (default_instance (reference "U") (unit 1) (value "TLP240A") (footprint "jacdac_access_switch_interface:LF1_TP1_TOSHIBA_11-5B201S"))
@@
     )
     (path "/00000000-0000-0000-0000-000060fd5ec1"
-      (reference "C1") (unit 1) (value "1uF, 10V") (footprint "jacdac_access_switch_interface:C_0402_1005Metric")
+      (reference "C1") (unit 1) (value "1uF") (footprint "jacdac_access_switch_interface:C_0402_1005Metric")
     )
     (path "/00000000-0000-0000-0000-000060fce670"
@@
     )
     (path "/00000000-0000-0000-0000-000060fdc132"
-      (reference "D1") (unit 1) (value "RCLAMP0521P-N") (footprint "jacdac_access_switch_interface:D_0402_1005Metric")
+      (reference "D1") (unit 1) (value "RCLAMP0521-P") (footprint "jacdac_access_switch_interface:D_0402_1005Metric")
     )
     (path "/00000000-0000-0000-0000-000060fdc147"
@@
     )
     (path "/5f7a3c9a-13e3-46f2-b2d2-95bfed512298"
-      (reference "J3") (unit 1) (value "pj313d") (footprint "jacdac_access_switch_interface:jack_3.5_pj313d_smt")
+      (reference "J3") (unit 1) (value "jack_3.5_pj313d") (footprint "jacdac_access_switch_interface:jack_3.5_pj313d_smt")
     )
     (path "/98c5c435-e865-46bd-a116-22aaef70c1b8"
@@
     )
     (path "/3e696000-af11-4a7a-bcc6-cf53a4befb15"
-      (reference "R13") (unit 1) (value "130") (footprint "jacdac_access_switch_interface:R_0402_1005Metric")
+      (reference "R13") (unit 1) (value "150") (footprint "jacdac_access_switch_interface:R_0402_1005Metric")
     )
     (path "/d076cc5d-8f0f-45de-94d1-1cd1ad649243"
